File: Electrique/Boost_Comm/Boost_Comm.sch (KiCad schematic (older format))
At the start: 23 parts, among them M1 CSD17571Q2, U1 TPS40210DGQ

Commit message: Traces pcb sans MOSFET
Parts:
- In_bus1: renamed from In_bus; footprint (none) -> TerminalBlock:TerminalBlock_bornier-2_P5.08mm
- Out_Bus1: renamed from Out_Bus; footprint (none) -> TerminalBlock:TerminalBlock_bornier-2_P5.08mm
Changed lines of the file:
@@
 Connection ~ 1700 5800
 $Comp
-L Connector:Screw_Terminal_01x02 In_bus
+L Connector:Screw_Terminal_01x02 In_bus1
 U 1 1 5EF4F93F
 P 1150 3550
-F 0 "In_bus" H 1230 3542 50  0000 L CNN
+F 0 "In_bus1" H 1230 3542 50  0000 L CNN
 F 1 "Screw_Terminal_01x02" H 1230 3451 50  0000 L CNN
-F 2 "" H 1150 3550 50  0001 C CNN
+F 2 "TerminalBlock:TerminalBlock_bornier-2_P5.08mm" H 1150 3550 50  0001 C CNN
 F 3 "~" H 1150 3550 50  0001 C CNN
 	1    1150 3550
@@
 $EndComp
 $Comp
-L Connector:Screw_Terminal_01x02 Out_Bus
+L Connector:Screw_Terminal_01x02 Out_Bus1
 U 1 1 5EF51525
 P 8950 5150
-F 0 "Out_Bus" H 9030 5142 50  0000 L CNN
+F 0 "Out_Bus1" H 9030 5142 50  0000 L CNN
 F 1 "Screw_Terminal_01x02" H 9030 5051 50  0000 L CNN
-F 2 "" H 8950 5150 50  0001 C CNN
+F 2 "TerminalBlock:TerminalBlock_bornier-2_P5.08mm" H 8950 5150 50  0001 C CNN
 F 3 "~" H 8950 5150 50  0001 C CNN
 	1    8950 5150

Commit message: Changement du footprint comm
Changement du footprint de m1 dans le convertisseur de communication
Parts:
- M1: footprint Boost_Comm:CSD17571Q2 -> Boost_Comm:7inch_SON_2x2_mm; symbol Device:Q_NMOS_DGS -> Boost_Comm-rescue:Custom_Boost_Comm_Q_NMOS_DGS_comm-Boost_Comm-cache
Connections:
- net at Riflt1.2, Rsense1.2: now also M1.4 (S); no longer M1.3 (S)
- net at Rg1.2: now also M1.3 (G); no longer M1.2 (G)
Changed lines of the file:
@@
 Wire Wire Line
 	5050 2850 5050 2350
-Connection ~ 6950 5100
 Connection ~ 6950 5800
 Wire Wire Line
@@
 Wire Wire Line
 	6950 5800 7550 5800
-$Comp
-L Device:Q_NMOS_DGS M1
-U 1 1 5E5F36EA
-P 6850 4450
-F 0 "M1" H 7054 4496 50  0000 L CNN
-F 1 "CSD17571Q2" H 7054 4405 50  0000 L CNN
-F 2 "Boost_Comm:CSD17571Q2" H 7050 4550 50  0001 C CNN
-F 3 "~" H 6850 4450 50  0001 C CNN
-	1    6850 4450
-	1    0    0    -1
-$EndComp
-Wire Wire Line
-	6950 4650 6950 5100
-Wire Wire Line
-	6650 4450 6550 4450
 $Comp
 L Device:C Coutx1
@@
 	7250 3350 7550 3350
 Wire Wire Line
-	7550 3350 7550 4700
-Wire Wire Line
-	7550 4700 8200 4700
-Wire Wire Line
 	8200 4700 8200 5000
-Connection ~ 7550 4700
 Wire Wire Line
 	7550 4700 7550 5000
@@
 Wire Wire Line
 	5750 2850 8200 2850
-Connection ~ 6950 3350
-Wire Wire Line
-	6950 4250 6950 3350
 Wire Wire Line
 	5750 3350 6950 3350
@@
 	1    0    0    -1
 $EndComp
+Connection ~ 7550 4700
+Wire Wire Line
+	7550 4700 8200 4700
+Wire Wire Line
+	7550 3350 7550 4700
+Connection ~ 6950 5100
+Connection ~ 6950 3350
+$Comp
+L Boost_Comm-rescue:Custom_Boost_Comm_Q_NMOS_DGS_comm-Boost_Comm-cache M1
+U 1 1 5E5F36EA
+P 6850 4450
+F 0 "M1" H 7054 4496 50  0000 L CNN
+F 1 "CSD17571Q2" H 7054 4405 50  0000 L CNN
+F 2 "Boost_Comm:7inch_SON_2x2_mm" H 7050 4550 50  0001 C CNN
+F 3 "https://www.ti.com/lit/ds/symlink/csd17571q2.pdf?ts=1605385207733&ref_url=https%253A%252F%252Fwww.ti.com%252Fproduct%252FCSD17571Q2%253FCMP%253Dconv-poasamples" H 6850 4450 50  0001 C CNN
+	1    6850 4450
+	1    0    0    -1
+$EndComp
+Wire Wire Line
+	6950 4650 6950 5100
+Wire Wire Line
+	6950 4250 6950 3350
+Wire Wire Line
+	6650 4450 6550 4450
 $EndSCHEMATC
